File: vctcxo-ref.kicad_pcb (KiCad board)
At the start: 2 copper layers, 57.2 x 27.9 mm, 18 parts, among them IC1 TPS79930, J1 CONN_01x02, J2 CONN_01x02, P1 COAX, P2 COAX, Y1 VCTCXO

Commit message: Tweaks.
Routing:
- net Net-(C4-Pad1): track 30.3 -> 119.2 mm, vias 0 -> 2
- net Net-(C5-Pad1): track 13.5 -> 16.0 mm
- net /V_3V0: track 39.1 -> 40.9 mm
Changed lines of the file:
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@@
-(kicad_pcb (version 20171130) (host pcbnew 5.1.2-f72e74a~84~ubuntu18.04.1)
+(kicad_pcb (version 20171130) (host pcbnew 5.1.3-ffb9f22~84~ubuntu18.04.1)
   (general
     (thickness 1.6)
     (drawings 29)
-    (tracks 69)
+    (tracks 114)
     (zones 0)
     (modules 18)
@@
   (segment (start 109.499713 115.805136) (end 109.469248 115.77323) (width 0.5) (layer F.Cu) (net 3))
   (segment (start 109.498953 115.838045) (end 109.499713 115.805136) (width 0.5) (layer F.Cu) (net 3))
-  (segment (start 110.49 114.046) (end 110.49 114.846998) (width 0.5) (layer F.Cu) (net 3))
   (segment (start 110.49 114.846998) (end 109.498953 115.838045) (width 0.5) (layer F.Cu) (net 3))
   (segment (start 95.4335 106.4965) (end 95.2305 106.4965) (width 0.5) (layer F.Cu) (net 3))
@@
   (segment (start 110.49 114.046) (end 110.49 108.966) (width 0.5) (layer F.Cu) (net 3))
   (segment (start 110.49 108.966) (end 105.156 103.632) (width 0.5) (layer F.Cu) (net 3))
+  (segment (start 127.565 124.43) (end 124.540001 121.405001) (width 0.5) (layer F.Cu) (net 3))
+  (segment (start 127.565 125.73) (end 127.565 124.43) (width 0.5) (layer F.Cu) (net 3))
+  (segment (start 124.540001 118.412352) (end 122.967648 116.84) (width 0.5) (layer F.Cu) (net 3))
+  (segment (start 124.540001 121.405001) (end 124.540001 118.412352) (width 0.5) (layer F.Cu) (net 3))
+  (segment (start 122.967648 116.84) (end 122.650148 116.5225) (width 0.5) (layer F.Cu) (net 3))
+  (segment (start 134.59 109.925) (end 131.565001 112.949999) (width 0.5) (layer F.Cu) (net 3))
+  (segment (start 135.89 109.925) (end 134.59 109.925) (width 0.5) (layer F.Cu) (net 3))
+  (segment (start 131.565001 112.949999) (end 130.81 112.949999) (width 0.5) (layer F.Cu) (net 3))
+  (segment (start 130.81 112.949999) (end 129.620001 112.949999) (width 0.5) (layer F.Cu) (net 3))
+  (segment (start 123.111353 112.949999) (end 122.861361 113.199991) (width 0.5) (layer F.Cu) (net 3))
+  (segment (start 129.620001 112.949999) (end 123.111353 112.949999) (width 0.5) (layer F.Cu) (net 3))
+  (segment (start 122.861361 113.199991) (end 120.638862 115.42249) (width 0.5) (layer F.Cu) (net 3))
+  (segment (start 120.638862 115.42249) (end 119.645139 115.42249) (width 0.5) (layer F.Cu) (net 3))
+  (segment (start 119.645139 115.42249) (end 115.950314 115.42249) (width 0.5) (layer F.Cu) (net 3))
+  (segment (start 118.815 124.43) (end 121.839999 121.405001) (width 0.5) (layer F.Cu) (net 3))
+  (segment (start 118.815 125.73) (end 118.815 124.43) (width 0.5) (layer F.Cu) (net 3))
+  (segment (start 121.839999 121.405001) (end 121.839999 118.823647) (width 0.5) (layer F.Cu) (net 3))
+  (segment (start 121.839999 118.823647) (end 121.523176 118.506824) (width 0.5) (layer F.Cu) (net 3))
+  (segment (start 121.523176 118.506824) (end 120.638862 117.62251) (width 0.5) (layer F.Cu) (net 3))
+  (segment (start 120.638862 117.62251) (end 119.38 117.62251) (width 0.5) (layer F.Cu) (net 3))
+  (segment (start 119.38 117.62251) (end 115.57 117.62251) (width 0.5) (layer F.Cu) (net 3))
+  (via (at 122.867384 116.517384) (size 0.8) (drill 0.4) (layers F.Cu B.Cu) (net 3))
+  (segment (start 122.650148 116.5225) (end 122.862268 116.5225) (width 0.5) (layer F.Cu) (net 3))
+  (segment (start 122.862268 116.5225) (end 122.867384 116.517384) (width 0.5) (layer F.Cu) (net 3))
+  (segment (start 134.59 118.675) (end 135.89 118.675) (width 0.5) (layer F.Cu) (net 3))
+  (segment (start 132.08 116.165) (end 134.59 118.675) (width 0.5) (layer F.Cu) (net 3))
+  (segment (start 122.650148 116.5225) (end 123.772638 115.40001) (width 0.5) (layer F.Cu) (net 3))
+  (segment (start 130.018499 115.480001) (end 130.188499 115.650001) (width 0.5) (layer F.Cu) (net 3))
+  (segment (start 123.772638 115.40001) (end 130.018499 115.40001) (width 0.5) (layer F.Cu) (net 3))
+  (segment (start 130.188499 115.650001) (end 132.08 115.650001) (width 0.5) (layer F.Cu) (net 3))
+  (segment (start 130.018499 115.40001) (end 130.018499 115.480001) (width 0.5) (layer F.Cu) (net 3))
+  (segment (start 132.08 115.650001) (end 132.08 116.165) (width 0.5) (layer F.Cu) (net 3))
+  (segment (start 108.852 115.989) (end 109.19 116.327) (width 0.5) (layer F.Cu) (net 3))
+  (segment (start 107.569 115.989) (end 108.852 115.989) (width 0.5) (layer F.Cu) (net 3))
+  (via (at 110.49 114.3) (size 0.8) (drill 0.4) (layers F.Cu B.Cu) (net 3))
+  (segment (start 110.49 114.3) (end 110.49 114.846998) (width 0.5) (layer F.Cu) (net 3))
+  (segment (start 110.49 114.046) (end 110.49 114.3) (width 0.5) (layer F.Cu) (net 3))
+  (segment (start 110.49 114.3) (end 112.776 116.586) (width 0.5) (layer B.Cu) (net 3))
+  (segment (start 112.776 116.586) (end 121.158 116.586) (width 0.5) (layer B.Cu) (net 3))
+  (segment (start 121.158 116.586) (end 121.158 116.332) (width 0.5) (layer B.Cu) (net 3))
+  (segment (start 121.158 116.332) (end 123.19 114.3) (width 0.5) (layer B.Cu) (net 3))
+  (segment (start 123.19 114.3) (end 131.572 114.3) (width 0.5) (layer B.Cu) (net 3))
   (segment (start 105.4735 105.3465) (end 100.7305 105.3465) (width 0.5) (layer F.Cu) (net 4))
   (segment (start 109.19 112.527) (end 109.19 109.063) (width 0.5) (layer F.Cu) (net 4))
   (segment (start 109.19 109.063) (end 105.4735 105.3465) (width 0.5) (layer F.Cu) (net 4))
+  (segment (start 109.19 112.768) (end 107.569 114.389) (width 0.5) (layer F.Cu) (net 4))
+  (segment (start 109.19 112.527) (end 109.19 112.768) (width 0.5) (layer F.Cu) (net 4))
   (segment (start 96.6805 113.223) (end 96.3955 113.223) (width 0.25) (layer F.Cu) (net 7))
   (segment (start 96.3955 113.223) (end 96.0755 112.903) (width 0.25) (layer F.Cu) (net 7))
@@
   (segment (start 102.743 111.633) (end 105.4735 108.9025) (width 0.5) (layer F.Cu) (net 8))
   (segment (start 99.6695 111.633) (end 102.743 111.633) (width 0.5) (layer F.Cu) (net 8))
+  (segment (start 112.1915 112.9285) (end 111.79 112.527) (width 0.5) (layer F.Cu) (net 8))
+  (segment (start 113.411 112.9285) (end 112.1915 112.9285) (width 0.5) (layer F.Cu) (net 8))
   (segment (start 112.9855 116.5225) (end 112.79 116.327) (width 0.5) (layer F.Cu) (net 9))
   (segment (start 112.79 116.327) (end 111.79 116.327) (width 0.5) (layer F.Cu) (net 9))

Commit message: Tweaks.
Parts:
- removed RV1: R_POT_TRIM, Potentiometer_SMD:Potentiometer_Vishay_TS53YL_Vertical
- added J3: CONN_01x01, TestPoint:TestPoint_THTPad_D1.5mm_Drill0.7mm, F.Cu at (94.0, 104.1)
- added J4: CONN_01x01, TestPoint:TestPoint_THTPad_D1.5mm_Drill0.7mm, F.Cu at (96.5, 106.7)
- added J5: CONN_01x01, TestPoint:TestPoint_THTPad_D1.5mm_Drill0.7mm, F.Cu at (99.1, 104.1)
- moved Y1 3.64 mm to (114.0, 115.2)
- moved C4 3.64 mm to (117.0, 114.5)
- moved C5 3.64 mm to (111.1, 116.0)
Connections:
- C4 pad 1: Net-(C4-Pad1) -> GND
- C5 pad 2: Net-(C4-Pad1) -> GND
- P1 pad 2: Net-(C4-Pad1) -> GND
- P2 pad 2: Net-(C4-Pad1) -> GND
- Y1 pad 2: Net-(C4-Pad1) -> GND
Routing:
- net Net-(C4-Pad1): track 119.2 -> 0.00 mm, vias 2 -> 0
- net GND: track 16.7 -> 71.2 mm, vias 5 -> 31
- net /V_3V0: track 40.9 -> 49.9 mm
- net Net-(C5-Pad1): track 16.0 -> 23.2 mm
- net /RF_OUT_TCXO: track 26.1 -> 22.7 mm
- net Net-(C7-Pad2): track 0.00 -> 2.95 mm
- net Net-(C6-Pad2): track 0.00 -> 2.95 mm
Other:
- outline, holes or cut-outs redrawn
- board text added: "+"
- board text added: "3.3V-5V"
- board text added: "40.00MHz"
- board text added: "LimeSDR VCTCXO"
- board text added: "Phil M0DNY"
- board text added: "r2019.08"
- board text removed: "VCTCXO Reference"

Commit message: Tweaks.
Parts:
- added C8: 100n, agg:0603, F.Cu at (73.9, 113.5)
- added C9: 2u2, agg:0603, F.Cu at (73.9, 116.0)
- added FB1: Ferrite_Bead_Small, agg:0603, F.Cu at (78.1, 113.5)
- added FB2: Ferrite_Bead_Small, agg:0603, F.Cu at (78.1, 116.0)
- added R1: 1K, agg:0603, F.Cu at (104.6, 101.9)
- added R2: 1K, agg:0603, F.Cu at (104.6, 104.1)
Connections:
- C1 pad 1: /VIN_5V -> Net-(C1-Pad1)
- IC1 pad 1: /VIN_5V -> Net-(C1-Pad1)
- IC1 pad 3: /VIN_5V -> Net-(C1-Pad1)
- J3 pad 1: /V_3V0 -> Net-(J3-Pad1)
- J5 pad 1: GND -> Net-(J5-Pad1)
Routing:
- net /V_3V0: track 49.9 -> 37.4 mm
- net Net-(J3-Pad1): track 0.00 -> 10.9 mm
- net GND: track 71.2 -> 64.9 mm
- net Net-(J5-Pad1): track 0.00 -> 4.79 mm
Other:
- board text added: "3.6V-6.5V"
- board text added: "~~0.1ppm/turn"
- board text removed: "3.3V-5V"

Commit message: Initial plot run.
Parts:
- moved C9 25.7 mm to (99.6, 114.8), turned to 90 degrees
- moved C8 22.3 mm to (96.0, 116.6), turned to 270 degrees
- moved FB2 19.7 mm to (97.8, 116.6), turned to 270 degrees
- moved FB1 19.0 mm to (97.0, 113.8), turned to 180 degrees
- moved C2 6.48 mm to (105.3, 117.9)
- moved C3 6.48 mm to (105.2, 112.9)
- moved IC1 6.48 mm to (104.3, 115.4)
- moved C1 6.45 mm to (101.2, 114.8)
Connections:
- C8 pad 2: GND -> Net-(C8-Pad2)
- FB2 pad 2: GND -> Net-(C8-Pad2)
- J1 pad 2: GND -> Net-(C8-Pad2)
- J2 pad 2: GND -> Net-(C8-Pad2)
Routing:
- net Net-(C8-Pad2): track 0.00 -> 23.2 mm, vias 0 -> 1
- net Net-(C1-Pad1): track 0.00 -> 12.3 mm, vias 0 -> 2
- net GND: track 64.9 -> 55.0 mm
- net /VIN_5V: track 30.6 -> 24.6 mm, vias 2 -> 0
- net /V_3V0: track 37.4 -> 33.3 mm
- net Net-(C5-Pad1): track 23.2 -> 24.2 mm
Other:
- outline, holes or cut-outs redrawn
- net class 50R: clearance 0.6 -> 0.2

Commit message: Sent to fab.
Other:
- board text added: "LimeRef Mini"
- board text removed: "LimeSDR VCTCXO"
Changed lines of the file:
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@@
   )
   (setup
-    (last_trace_width 0.75)
+    (last_trace_width 0.25)
     (user_trace_width 0.5)
     (user_trace_width 0.75)
@@
     )
   )
-  (gr_text ~~0.1ppm/turn (at 100.838 109.22) (layer F.SilkS)
-    (effects (font (size 1.2 1.2) (thickness 0.3)))
+  (gr_text ~~0.1ppm/turn (at 96.52 109.22) (layer F.SilkS)
+    (effects (font (size 1 1) (thickness 0.2)))
   )
   (gr_text + (at 82.55 112.7125) (layer F.SilkS)
@@
     (effects (font (size 1.5 1.5) (thickness 0.3)))
   )
-  (gr_text 40.00MHz (at 114.554 121.412) (layer F.SilkS)
+  (gr_text 40.00MHz (at 113.8555 121.285) (layer F.SilkS)
     (effects (font (size 1.5 1.5) (thickness 0.3)))
   )
-  (gr_text r2019.08 (at 130.302 105.156) (layer F.SilkS)
+  (gr_text r2019.08 (at 130.175 105.9815) (layer F.SilkS)
     (effects (font (size 1 1) (thickness 0.2)) (justify right))
   )
-  (gr_text "Phil M0DNY" (at 130.302 107.95) (layer F.SilkS)
+  (gr_text "Phil M0DNY" (at 130.2385 108.966) (layer F.SilkS)
     (effects (font (size 1.5 1.5) (thickness 0.25) italic) (justify right))
   )
@@
   (gr_line (start 110.236 117.602) (end 110.236 112.776) (layer Edge.Cuts) (width 0.05))
   (gr_line (start 118.364 118.237) (end 110.871 118.237) (layer Edge.Cuts) (width 0.05))
-  (gr_text "LimeSDR VCTCXO" (at 130.302 102.362) (layer F.SilkS)
-    (effects (font (size 1.5 1.5) (thickness 0.3)) (justify right))
+  (gr_text "LimeRef Mini" (at 130.175 102.9335) (layer F.SilkS)
+    (effects (font (size 2 2) (thickness 0.4)) (justify right))
   )
   (gr_arc (start 85.09 104.14) (end 85.09 100.33) (angle -90) (layer Edge.Cuts) (width 0.05))
@@
   (via (at 100.965 117.221) (size 0.8) (drill 0.4) (layers F.Cu B.Cu) (net 1))
   (segment (start 99.568 115.608) (end 101.1555 115.608) (width 0.75) (layer F.Cu) (net 1))
-  (segment (start 97.79 117.386) (end 96.012 117.386) (width 0.75) (layer F.Cu) (net 12))
   (segment (start 105.5425 116.481) (end 105.6305 116.393) (width 0.75) (layer F.Cu) (net 2))
   (segment (start 105.6305 117.69) (end 105.7965 117.856) (width 0.25) (layer F.Cu) (net 2))
@@
   (segment (start 132.9435 114.3) (end 135.89 114.3) (width 0.75) (layer F.Cu) (net 4))
   (segment (start 123.19 122.7835) (end 123.19 125.73) (width 0.75) (layer F.Cu) (net 5))
-  (segment (start 103.0305 114.493) (end 102.7455 114.493) (width 0.75) (layer F.Cu) (net 11))
-  (segment (start 102.7455 114.493) (end 102.4255 114.173) (width 0.75) (layer F.Cu) (net 11))
-  (via (at 102.9335 113.284014) (size 0.8) (drill 0.4) (layers F.Cu B.Cu) (net 11))
-  (via (at 102.933506 117.475) (size 0.8) (drill 0.4) (layers F.Cu B.Cu) (net 11))
-  (segment (start 102.9335 117.474994) (end 102.933506 117.475) (width 0.75) (layer B.Cu) (net 11))
-  (segment (start 102.9335 113.284014) (end 102.9335 117.474994) (width 0.75) (layer B.Cu) (net 11))
-  (segment (start 103.0305 117.378006) (end 102.933506 117.475) (width 0.75) (layer F.Cu) (net 11))
-  (segment (start 103.0305 116.393) (end 103.0305 117.378006) (width 0.75) (layer F.Cu) (net 11))
-  (segment (start 102.935501 114.173) (end 103.0305 114.267999) (width 0.75) (layer F.Cu) (net 11))
-  (segment (start 101.1555 114.173) (end 102.935501 114.173) (width 0.75) (layer F.Cu) (net 11))
-  (segment (start 102.9335 114.170999) (end 102.935501 114.173) (width 0.75) (layer F.Cu) (net 11))
-  (segment (start 102.9335 113.284014) (end 102.9335 114.170999) (width 0.75) (layer F.Cu) (net 11))
   (segment (start 96.012 114.008) (end 96.228 113.792) (width 0.75) (layer F.Cu) (net 6))
   (segment (start 96.012 115.786) (end 96.012 114.008) (width 0.75) (layer F.Cu) (net 6))
@@
   (segment (start 100.33 104.14) (end 99.06 104.14) (width 0.75) (layer F.Cu) (net 10))
   (segment (start 100.33 104.14) (end 103.848 104.14) (width 0.75) (layer F.Cu) (net 10))
+  (segment (start 103.0305 114.493) (end 102.7455 114.493) (width 0.75) (layer F.Cu) (net 11))
+  (segment (start 102.7455 114.493) (end 102.4255 114.173) (width 0.75) (layer F.Cu) (net 11))
+  (via (at 102.9335 113.284014) (size 0.8) (drill 0.4) (layers F.Cu B.Cu) (net 11))
+  (via (at 102.933506 117.475) (size 0.8) (drill 0.4) (layers F.Cu B.Cu) (net 11))
+  (segment (start 102.9335 117.474994) (end 102.933506 117.475) (width 0.75) (layer B.Cu) (net 11))
+  (segment (start 102.9335 113.284014) (end 102.9335 117.474994) (width 0.75) (layer B.Cu) (net 11))
+  (segment (start 103.0305 117.378006) (end 102.933506 117.475) (width 0.75) (layer F.Cu) (net 11))
+  (segment (start 103.0305 116.393) (end 103.0305 117.378006) (width 0.75) (layer F.Cu) (net 11))
+  (segment (start 102.935501 114.173) (end 103.0305 114.267999) (width 0.75) (layer F.Cu) (net 11))
+  (segment (start 101.1555 114.173) (end 102.935501 114.173) (width 0.75) (layer F.Cu) (net 11))
+  (segment (start 102.9335 114.170999) (end 102.935501 114.173) (width 0.75) (layer F.Cu) (net 11))
+  (segment (start 102.9335 113.284014) (end 102.9335 114.170999) (width 0.75) (layer F.Cu) (net 11))
   (segment (start 99.568 114.008) (end 101.1555 114.008) (width 0.75) (layer F.Cu) (net 11))
   (segment (start 99.352 113.792) (end 99.568 114.008) (width 0.75) (layer F.Cu) (net 11))
   (segment (start 97.828 113.792) (end 99.352 113.792) (width 0.75) (layer F.Cu) (net 11))
+  (segment (start 97.79 117.386) (end 96.012 117.386) (width 0.75) (layer F.Cu) (net 12))
   (segment (start 94.488 124.714) (end 94.488 120.396) (width 0.75) (layer B.Cu) (net 12))
   (segment (start 94.488 120.396) (end 96.012 118.872) (width 0.75) (layer B.Cu) (net 12))
